File: Hardware/Bicycle_V2.kicad_pcb (KiCad board)
At the start: 2 copper layers, 95 x 48.8 mm, 32 parts, among them J1 SENSOR, J2 SWD, J3 BLUETOOTH Module, J4 Switch, U1 STM32L011K4T6, U2 LD3985M33R_SOT23

Commit message: Latest Release
Parts:
- removed BZ1: Buzzer, Buzzer_Beeper:Buzzer_12x9.5RM7.6
- removed FB1: 120R, Inductor_SMD:L_0805_2012Metric
- removed J3: BLUETOOTH Module, Connector_PinHeader_2.54mm:PinHeader_1x04_P2.54mm_Horizontal
- added J5: Conn_01x03_Pin, Connector_PinHeader_2.54mm:PinHeader_1x03_P2.54mm_Vertical, F.Cu at (119.3, 59.7)
- added J7: Conn_01x08_Socket, Connector_PinSocket_2.54mm:PinSocket_1x08_P2.54mm_Vertical, F.Cu at (157.8, 59.7)
- added R5: 10k, Resistor_SMD:R_0805_2012Metric, B.Cu at (116.1, 58.8)
- moved R11 12.0 mm to (135.1, 52.8)
- moved R12 11.9 mm to (132.9, 52.8)
- moved J4 7.82 mm to (166.2, 57.1), turned to 0 degrees
- moved R1 5.04 mm to (116.1, 63.9)
- moved C7 2.01 mm to (128.9, 53.6), turned to 0 degrees
- moved C5 2.01 mm to (128.9, 58.1)
- moved C6 2.01 mm to (128.9, 55.9)
Connections:
- C5 pad 1: Net-(C5-Pad1) -> +3.3V
- C6 pad 1: Net-(C5-Pad1) -> +3.3V
- R1 pad 1: /BOOT0 -> Net-(J5-Pin_3)
- U1 pad 10: /ADC_IN -> /BackLight
- U1 pad 11: unconnected-(U1-Pad11) -> /SPI1_SCK
- U1 pad 13: unconnected-(U1-Pad13) -> /SPI1_MOSI
- U1 pad 28: /Buzzer -> unconnected-(U1-PB5-Pad28)
- U1 pad 31: /BOOT0 -> Net-(J5-Pin_2)
- U1 pad 5: Net-(C5-Pad1) -> +3.3V
- U1 pad 6: unconnected-(U1-Pad6) -> /ADC_IN
- U1 pad 7: unconnected-(U1-Pad7) -> /RST
- U1 pad 8: /USART_TX -> /CS
- U1 pad 9: /USART_RX -> /DC
Routing:
- net /RST: track 0.00 -> 35.3 mm
- net /CS: track 0.00 -> 30.6 mm
- net +3.3V: track 214.9 -> 242.3 mm, vias 0 -> 1
- net /DC: track 0.00 -> 27.0 mm
- net /SPI1_MOSI: track 0.00 -> 23.8 mm
- net /SPI1_SCK: track 0.00 -> 19.9 mm
- net /BackLight: track 0.00 -> 15.3 mm
- net /USART_TX: track 14.2 -> 0.00 mm
- net VBUS: track 49.5 -> 63.6 mm
- net /USART_RX: track 13.0 -> 0.00 mm
- net /Buzzer: track 8.86 -> 0.00 mm
- net Net-(C5-Pad1): track 7.37 -> 0.00 mm
- net Net-(BT1-+): track 13.4 -> 20.3 mm
- net /ADC_IN: track 7.36 -> 14.0 mm
- net Net-(J5-Pin_2): track 0.00 -> 5.95 mm
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- added copper zone on F.Cu, net GND
