File: Hardware/Bicycle_V2.kicad_sch (KiCad schematic)
At the start: 32 parts, among them J1 SENSOR, J2 SWD, J3 BLUETOOTH Module, J4 Switch, U1 STM32L011K4T6, U2 LD3985M33R_SOT23

Commit message: Latest Release
Parts:
- removed BZ1: Buzzer, Buzzer_Beeper:Buzzer_12x9.5RM7.6, symbol Device:Buzzer
- removed FB1: 120R, Inductor_SMD:L_0805_2012Metric, symbol Device:FerriteBead
- removed J3: BLUETOOTH Module, Connector_PinHeader_2.54mm:PinHeader_1x04_P2.54mm_Horizontal, symbol Connector:Conn_01x04_Female
- added J5: Conn_01x03_Pin, Connector_PinHeader_2.54mm:PinHeader_1x03_P2.54mm_Vertical, symbol Connector:Conn_01x03_Pin
- added J7: Conn_01x08_Socket, Connector_PinSocket_2.54mm:PinSocket_1x08_P2.54mm_Vertical, symbol Connector:Conn_01x08_Socket
- added R5: 10k, Resistor_SMD:R_0805_2012Metric, symbol Device:R
Connections:
- net +3.3V: now also C5.1, C6.1, U1.5 (VDDA), J7.6 (Pin_6), R5.2
- net ADC_IN: now also U1.6 (PA0); no longer U1.10 (PA4)
- net BOOT0: no longer R1.1, U1.31 (PB9)
- net GND: now also J7.8 (Pin_8)
- net SPI1_SCK: now reaches U1.11 (PA5)
- net SPI1_SCK: now also J7.5 (Pin_5)
- net SPI1_MOSI: now reaches U1.13 (PA7)
- net SPI1_MOSI: now also J7.4 (Pin_4)
- net RST: now reaches U1.7 (PA1)
- net RST: now also J7.1 (Pin_1)
- net Buzzer: no longer names the net of U1.28 (PB5)
- net USART_RX renamed DC
- net DC: now also J7.3 (Pin_3)
- net USART_TX renamed CS
- net CS: now also J7.2 (Pin_2)
- new net: J5.3 (Pin_3), R1.1
- new net: J5.1 (Pin_1), R5.1
- new net: J5.2 (Pin_2), U1.31 (PB9)
- new net BackLight: J7.7 (Pin_7), U1.10 (PA4)
Other:
- note added: "For Changing The BOOT config"
- moved on the sheet: R1
